File: mainboard.brd (EAGLE design)
At the start: 100 x 80 mm, 21 parts

Commit message: pcb
Parts:
- moved PROG 111.0 mm to (36.1, 38.2), turned to 90 degrees
- moved EDF 63.6 mm to (1.78, 10.3), turned to 90 degrees
- moved DRV 61.5 mm to (19.6, 10.3)
- moved EN 60.3 mm to (5.59, 45.8), turned to 180 degrees
- moved M2 59.1 mm to (6.86, 2.67), turned to 90 degrees
- moved R5 58.8 mm to (5.59, 40.8), turned to 90 degrees
- moved QTRPWR 50.5 mm to (1.78, 17.9), turned to 90 degrees
- moved M1 50.2 mm to (6.86, 9.02), turned to 270 degrees
- moved BAT 41.4 mm to (6.86, 15.4), turned to 90 degrees
- moved ACT 35.5 mm to (32.3, 39.5), turned to 180 degrees
- moved C2 31.8 mm to (33.5, 15.7), turned to 180 degrees
- moved FLASH 30.8 mm to (36.1, 26.8), turned to 90 degrees
- moved R3 29.1 mm to (32.3, 43.3), turned to 270 degrees
- moved R1 28.7 mm to (32.3, 21.7), turned to 90 degrees
- moved QTRIO 28.3 mm to (1.78, 31.9), turned to 90 degrees
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Routing:
- net +3V3: track 0.00 -> 113.7 mm
- net QTR8: track 0.00 -> 45.1 mm, vias 0 -> 1
- net M2B: track 0.00 -> 40.3 mm, vias 0 -> 1
- net M2E: track 0.00 -> 37.0 mm, vias 0 -> 1
- net M2A: track 0.00 -> 36.2 mm, vias 0 -> 1
- net EDF: track 0.00 -> 35.9 mm, vias 0 -> 1
- net +5V: track 0.00 -> 30.3 mm
- net M1A: track 0.00 -> 21.5 mm, vias 0 -> 1
- net M1B: track 0.00 -> 19.7 mm, vias 0 -> 1
- net EN: track 0.00 -> 16.5 mm
- net +12V: track 0.00 -> 16.1 mm
- net QTR1: track 0.00 -> 15.4 mm
- net M1E: track 0.00 -> 13.3 mm, vias 0 -> 1
- net QTR7: track 0.00 -> 12.0 mm
- net QTR6: track 0.00 -> 11.5 mm
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Other:
- board size 100 x 80 mm -> 39 x 49.5 mm
- board text added: "+"
- board text added: "-"
- board text added: "1"
- board text added: "B"
- board text added: "L"
- board text added: "R"
- board text added: "T"
